File: boardpov.brd (EAGLE design)
At the start: 225 x 38 mm, 40 parts

Commit message: sdsd
Parts:
- added C1: (no value), adafruit:C025-025X050
- added JP1: (no value), pinhead:1X03
- added JP2, JP5: (no value), adafruit:1X06-CLEANBIG
Connections:
- new net N$1: U$10.GND-, U$11.GND-, U$12.GND-, U$13.GND-, U$14.GND-, U$15.GND-, U$16.GND-, U$17.GND-, U$18.GND-, U$19.GND-, U$2.GND-, U$20.GND-, U$21.GND-, U$22.GND-, U$23.GND-, U$24.GND-, U$25.GND-, U$26.GND-, U$27.GND-, U$28.GND-, U$29.GND-, U$3.GND-, U$30.GND-, U$31.GND-, U$4.GND-, U$41.GND-, U$42.GND-, U$43.GND-, U$44.GND-, U$45.GND-, U$46.GND-, U$47.GND-, U$48.GND-, U$5.GND-, U$6.GND-, U$7.GND-, U$8.GND-, U$9.GND-
- new net N$2: U$1.21, U$48.GND, U$49.GND, U$49.GND-
- new net N$3: U$45.VDD, U$45.VDD+, U$46.VDD, U$46.VDD+, U$47.VDD, U$47.VDD+, U$48.VDD, U$49.VDD
- net GND: no longer U$1.21
Changed lines of the file:
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@@
 <layer number="112" name="tSilk" color="7" fill="1" visible="yes" active="yes"/>
 <layer number="113" name="LOGO" color="7" fill="1" visible="yes" active="yes"/>
+<layer number="114" name="Badge_Outline" color="7" fill="1" visible="yes" active="yes"/>
+<layer number="115" name="ReferenceISLANDS" color="7" fill="1" visible="yes" active="yes"/>
 <layer number="116" name="Patch_BOT" color="9" fill="4" visible="yes" active="yes"/>
+<layer number="118" name="Rect_Pads" color="7" fill="1" visible="yes" active="yes"/>
 <layer number="121" name="_tsilk" color="7" fill="1" visible="yes" active="yes"/>
 <layer number="122" name="_bsilk" color="7" fill="1" visible="yes" active="yes"/>
@@
 <layer number="223" name="223bmp" color="24" fill="1" visible="no" active="no"/>
 <layer number="224" name="224bmp" color="25" fill="1" visible="no" active="no"/>
+<layer number="225" name="225bmp" color="7" fill="1" visible="yes" active="yes"/>
+<layer number="226" name="226bmp" color="7" fill="1" visible="yes" active="yes"/>
+<layer number="227" name="227bmp" color="7" fill="1" visible="yes" active="yes"/>
+<layer number="228" name="228bmp" color="7" fill="1" visible="yes" active="yes"/>
+<layer number="229" name="229bmp" color="7" fill="1" visible="yes" active="yes"/>
+<layer number="230" name="230bmp" color="7" fill="1" visible="yes" active="yes"/>
+<layer number="231" name="231bmp" color="7" fill="1" visible="yes" active="yes"/>
+<layer number="232" name="Eagle3D_PG2" color="7" fill="1" visible="yes" active="yes"/>
+<layer number="233" name="Eagle3D_PG3" color="7" fill="1" visible="yes" active="yes"/>
 <layer number="248" name="Housing" color="7" fill="1" visible="yes" active="yes"/>
 <layer number="249" name="Edge" color="7" fill="1" visible="yes" active="yes"/>
@@
 <layer number="251" name="SMDround" color="7" fill="1" visible="no" active="no"/>
 <layer number="254" name="cooling" color="7" fill="1" visible="yes" active="yes"/>
+<layer number="255" name="routoute" color="7" fill="1" visible="yes" active="yes"/>
 </layers>
 <board>
@@
 <element name="U$48" library="POVPARTS" package="APA102-2020" value="APA102-202020-20" x="53.4" y="17.3"/>
 <element name="U$49" library="POVPARTS" package="APA102-2020" value="APA102-202020-20" x="48.9" y="17.3"/>
+<element name="JP1" library="pinhead" library_urn="urn:adsk.eagle:library:325" package="1X03" package3d_urn="urn:adsk.eagle:package:22458/2" value="" x="219.7" y="30.5" rot="R270"/>
+<element name="JP2" library="adafruit" package="1X06-CLEANBIG" value="" x="213.6355625" y="13.03554375" rot="R180"/>
+<element name="JP5" library="adafruit" package="1X06-CLEANBIG" value="" x="213.6355625" y="23.19554375" rot="R180"/>
+<element name="C1" library="adafruit" library_urn="urn:adsk.eagle:library:420" package="C025-025X050" value="" x="220.2" y="5.4" rot="R90"/>
 </elements>
 <signals>
@@
 <signal name="GND">
 <contactref element="U$1" pad="2"/>
-<contactref element="U$1" pad="21"/>
-<wire x1="11.362" y1="10.16" x2="16.442" y2="27.94" width="0" layer="19" extent="1-1"/>
 </signal>
 <signal name="3V3">
@@
 <signal name="VBAT">
 <contactref element="U$1" pad="22"/>
+</signal>
+<signal name="N$1">
+<contactref element="U$48" pad="GND-"/>
+<contactref element="U$47" pad="GND-"/>
+<contactref element="U$46" pad="GND-"/>
+<contactref element="U$45" pad="GND-"/>
+<contactref element="U$44" pad="GND-"/>
+<contactref element="U$31" pad="GND-"/>
+<contactref element="U$30" pad="GND-"/>
+<contactref element="U$29" pad="GND-"/>
+<contactref element="U$28" pad="GND-"/>
+<contactref element="U$27" pad="GND-"/>
+<contactref element="U$26" pad="GND-"/>
+<contactref element="U$25" pad="GND-"/>
+<contactref element="U$24" pad="GND-"/>
+<contactref element="U$23" pad="GND-"/>
+<contactref element="U$22" pad="GND-"/>
+<contactref element="U$21" pad="GND-"/>
+<contactref element="U$20" pad="GND-"/>
+<contactref element="U$19" pad="GND-"/>
+<contactref element="U$18" pad="GND-"/>
+<contactref element="U$17" pad="GND-"/>
+<contactref element="U$16" pad="GND-"/>
+<contactref element="U$15" pad="GND-"/>
+<contactref element="U$14" pad="GND-"/>
+<contactref element="U$13" pad="GND-"/>
+<contactref element="U$12" pad="GND-"/>
+<contactref element="U$11" pad="GND-"/>
+<contactref element="U$10" pad="GND-"/>
+<contactref element="U$9" pad="GND-"/>
+<contactref element="U$8" pad="GND-"/>
+<contactref element="U$7" pad="GND-"/>
+<contactref element="U$6" pad="GND-"/>
+<contactref element="U$5" pad="GND-"/>
+<contactref element="U$4" pad="GND-"/>
+<contactref element="U$3" pad="GND-"/>
+<contactref element="U$2" pad="GND-"/>
+<contactref element="U$41" pad="GND-"/>
+<contactref element="U$42" pad="GND-"/>
+<contactref element="U$43" pad="GND-"/>
+<wire x1="216.67" y1="18" x2="221.17" y2="18" width="0" layer="19" extent="1-1"/>
+<wire x1="212.17" y1="18" x2="216.67" y2="18" width="0" layer="19" extent="1-1"/>
+<wire x1="207.67" y1="18" x2="212.17" y2="18" width="0" layer="19" extent="1-1"/>
+<wire x1="203.17" y1="18" x2="207.67" y2="18" width="0" layer="19" extent="1-1"/>
+<wire x1="198.67" y1="18" x2="203.17" y2="18" width="0" layer="19" extent="1-1"/>
+<wire x1="194.17" y1="18" x2="198.67" y2="18" width="0" layer="19" extent="1-1"/>
+<wire x1="189.67" y1="18" x2="194.17" y2="18" width="0" layer="19" extent="1-1"/>
+<wire x1="185.17" y1="18" x2="189.67" y2="18" width="0" layer="19" extent="1-1"/>
+<wire x1="180.67" y1="18" x2="185.17" y2="18" width="0" layer="19" extent="1-1"/>
+<wire x1="176.17" y1="18" x2="180.67" y2="18" width="0" layer="19" extent="1-1"/>
+<wire x1="171.67" y1="18" x2="176.17" y2="18" width="0" layer="19" extent="1-1"/>
+<wire x1="167.17" y1="18" x2="171.67" y2="18" width="0" layer="19" extent="1-1"/>
+<wire x1="162.67" y1="18" x2="167.17" y2="18" width="0" layer="19" extent="1-1"/>
+<wire x1="158.17" y1="18" x2="162.67" y2="18" width="0" layer="19" extent="1-1"/>
+<wire x1="153.67" y1="18" x2="158.17" y2="18" width="0" layer="19" extent="1-1"/>
+<wire x1="149.17" y1="18" x2="153.67" y2="18" width="0" layer="19" extent="1-1"/>
+<wire x1="144.67" y1="18" x2="149.17" y2="18" width="0" layer="19" extent="1-1"/>
+<wire x1="140.17" y1="18" x2="144.67" y2="18" width="0" layer="19" extent="1-1"/>
+<wire x1="135.67" y1="18" x2="140.17" y2="18" width="0" layer="19" extent="1-1"/>
+<wire x1="131.17" y1="18" x2="135.67" y2="18" width="0" layer="19" extent="1-1"/>
+<wire x1="126.67" y1="18" x2="131.17" y2="18" width="0" layer="19" extent="1-1"/>
+<wire x1="122.17" y1="18" x2="126.67" y2="18" width="0" layer="19" extent="1-1"/>
+<wire x1="117.67" y1="18" x2="122.17" y2="18" width="0" layer="19" extent="1-1"/>
+<wire x1="113.17" y1="18" x2="117.67" y2="18" width="0" layer="19" extent="1-1"/>
+<wire x1="108.67" y1="18" x2="113.17" y2="18" width="0" layer="19" extent="1-1"/>
+<wire x1="104.17" y1="18" x2="108.67" y2="18" width="0" layer="19" extent="1-1"/>
+<wire x1="99.67" y1="18" x2="104.17" y2="18" width="0" layer="19" extent="1-1"/>
+<wire x1="95.17" y1="18" x2="99.67" y2="18" width="0" layer="19" extent="1-1"/>
+<wire x1="90.67" y1="18" x2="95.17" y2="18" width="0" layer="19" extent="1-1"/>
+<wire x1="86.17" y1="18" x2="90.67" y2="18" width="0" layer="19" extent="1-1"/>
+<wire x1="81.67" y1="18" x2="86.17" y2="18" width="0" layer="19" extent="1-1"/>
+<wire x1="77.17" y1="18" x2="81.67" y2="18" width="0" layer="19" extent="1-1"/>
+<wire x1="72.67" y1="18" x2="77.17" y2="18" width="0" layer="19" extent="1-1"/>
+<wire x1="68.17" y1="18" x2="72.67" y2="18" width="0" layer="19" extent="1-1"/>
+<wire x1="63.67" y1="18" x2="68.17" y2="18" width="0" layer="19" extent="1-1"/>
+<wire x1="59.17" y1="18" x2="63.67" y2="18" width="0" layer="19" extent="1-1"/>
+<wire x1="54.67" y1="18" x2="59.17" y2="18" width="0" layer="19" extent="1-1"/>
+</signal>
+<signal name="N$2">
+<contactref element="U$1" pad="21"/>
+<contactref element="U$49" pad="GND"/>
+<contactref element="U$49" pad="GND-"/>
+<contactref element="U$48" pad="GND"/>
+<wire x1="50.17" y1="18" x2="53.8" y2="19.44" width="0" layer="19" extent="1-16"/>
+<wire x1="49.3" y1="19.44" x2="50.17" y2="18" width="0" layer="19" extent="1-16"/>
+<wire x1="16.442" y1="27.94" x2="49.3" y2="19.44" width="0" layer="19" extent="16-16"/>
+</signal>
+<signal name="N$3">
+<contactref element="U$49" pad="VDD"/>
+<contactref element="U$48" pad="VDD"/>
+<contactref element="U$47" pad="VDD+"/>
+<contactref element="U$47" pad="VDD"/>
+<contactref element="U$46" pad="VDD+"/>
+<contactref element="U$46" pad="VDD"/>
+<contactref element="U$45" pad="VDD+"/>
+<contactref element="U$45" pad="VDD"/>
+<wire x1="68.17" y1="19.44" x2="69.04" y2="19.44" width="0" layer="19" extent="1-16"/>
+<wire x1="64.54" y1="19.44" x2="68.17" y2="19.44" width="0" layer="19" extent="1-16"/>
+<wire x1="63.67" y1="19.44" x2="64.54" y2="19.44" width="0" layer="19" extent="1-16"/>
+<wire x1="60.04" y1="19.44" x2="63.67" y2="19.44" width="0" layer="19" extent="1-16"/>
+<wire x1="59.17" y1="19.44" x2="60.04" y2="19.44" width="0" layer="19" extent="1-16"/>
+<wire x1="55.54" y1="19.44" x2="59.17" y2="19.44" width="0" layer="19" extent="1-16"/>
+<wire x1="51.04" y1="19.44" x2="55.54" y2="19.44" width="0" layer="19" extent="16-16"/>
 </signal>
 </signals>
@@
 which will not be processed correctly with this version.
 </note>
+<note version="8.2" severity="warning">
+Since Version 8.2, EAGLE supports online libraries. The ids
+of those online libraries will not be understood (or retained)
+with this version.
+</note>
+<note version="8.3" severity="warning">
+Since Version 8.3, EAGLE supports URNs for individual library
+assets (packages, symbols, and devices). The URNs of those assets
+will not be understood (or retained) with this version.
+</note>
+<note version="8.3" severity="warning">
+Since Version 8.3, EAGLE supports the association of 3D packages
+with devices in libraries, schematics, and board files. Those 3D
+packages will not be understood (or retained) with this version.
+</note>
 </compatibility>

Commit message: sd
Parts:
- added J1: (no value), SparkFun-Connectors:1X02
Connections:
- removed net GND: U$1.2
- removed net VIN: U$1.1
- new net N$10: U$45.CKL, U$46.CK0
- new net N$11: U$45.SD1, U$46.SD0
- new net N$12: U$44.CKL, U$45.CK0
- new net N$13: U$44.SD1, U$45.SD0
- new net N$14: U$26.SD1, U$44.SD0
- new net N$15: U$26.CKL, U$44.CK0
- new net N$16: U$26.SD0, U$27.SD1
- new net N$17: U$26.CK0, U$27.CKL
- new net N$18: U$27.CK0, U$28.CKL
- new net N$19: U$27.SD0, U$28.SD1
- new net N$20: U$28.CK0, U$29.CKL
- new net N$21: U$28.SD0, U$29.SD1
- new net N$22: U$29.CK0, U$30.CKL
- new net N$23: U$29.SD0, U$30.SD1
- new net N$24: U$30.SD0, U$31.SD1
- new net N$25: U$30.CK0, U$31.CKL
- new net N$26: U$25.SD1, U$31.SD0
- new net N$27: U$25.CKL, U$31.CK0
- new net N$28: U$20.CKL, U$21.CK0
- new net N$29: U$20.SD1, U$21.SD0
- new net N$30: U$21.SD1, U$22.SD0
- new net N$31: U$21.CKL, U$22.CK0
- new net N$32: U$22.CKL, U$23.CK0
- new net N$33: U$22.SD1, U$23.SD0
- new net N$34: U$23.SD1, U$24.SD0
- new net N$35: U$23.CKL, U$24.CK0
- new net N$36: U$24.CKL, U$25.CK0
- new net N$37: U$24.SD1, U$25.SD0
- new net N$38: U$14.SD1, U$20.CK0
- new net N$39: U$14.CKL, U$20.SD0
- new net N$4: U$48.SD1, U$49.SD0
- new net N$40: U$14.CK0, U$15.CKL
- new net N$41: U$14.SD0, U$15.SD1
- new net N$42: U$15.CK0, U$16.CKL
- new net N$43: U$15.SD0, U$16.SD1
- new net N$44: U$16.CK0, U$17.CKL
- new net N$45: U$16.SD0, U$17.SD1
- new net N$46: U$17.CK0, U$18.CKL
- new net N$47: U$17.SD0, U$18.SD1
- new net N$48: U$18.CK0, U$19.CKL
- new net N$49: U$18.SD0, U$19.SD1
- new net N$5: U$48.CKL, U$49.CK0
- new net N$50: U$13.SD1, U$19.SD0
- new net N$51: U$13.CKL, U$19.CK0
- new net N$52: U$8.CKL, U$9.CK0
- new net N$53: U$8.SD1, U$9.SD0
- new net N$54: U$10.SD0, U$9.SD1
- new net N$55: U$10.CK0, U$9.CKL
- new net N$56: U$10.CKL, U$11.CK0
- new net N$57: U$10.SD1, U$11.SD0
- new net N$58: U$11.SD1, U$12.SD0
- new net N$59: U$11.CKL, U$12.CK0
- new net N$6: U$47.CKL, U$48.CK0
- new net N$7: U$47.SD1, U$48.SD0
- new net N$8: U$46.SD1, U$47.SD0
- new net N$9: U$46.CKL, U$47.CK0
- net N$1: now also J1.2, U$1.1; no longer U$10.GND-, U$11.GND-, U$12.GND-, U$13.GND-, U$14.GND-, U$15.GND-, U$16.GND-, U$17.GND-, U$18.GND-, U$19.GND-, U$2.GND-, U$20.GND-, U$21.GND-, U$22.GND-, U$23.GND-, U$24.GND-, U$25.GND-, U$26.GND-, U$27.GND-, U$28.GND-, U$29.GND-, U$3.GND-, U$30.GND-, U$31.GND-, U$4.GND-, U$41.GND-, U$42.GND-, U$43.GND-, U$44.GND-, U$45.GND-, U$46.GND-, U$47.GND-, U$48.GND-, U$5.GND-, U$6.GND-, U$7.GND-, U$8.GND-, U$9.GND-
- net N$2: now also J1.1, U$1.2, U$10.GND, U$10.GND-, U$11.GND, U$11.GND-, U$12.GND, U$12.GND-, U$13.GND, U$13.GND-, U$14.GND, U$14.GND-, U$15.GND, U$15.GND-, U$16.GND, U$16.GND-, U$17.GND, U$17.GND-, U$18.GND, U$18.GND-, U$19.GND, U$19.GND-, U$2.GND, U$2.GND-, U$20.GND, U$20.GND-, U$21.GND, U$21.GND-, U$22.GND, U$22.GND-, U$23.GND, U$23.GND-, U$24.GND, U$24.GND-, U$25.GND, U$25.GND-, U$26.GND, U$26.GND-, U$27.GND, U$27.GND-, U$28.GND, U$28.GND-, U$29.GND, U$29.GND-, U$3.GND, U$3.GND-, U$30.GND, U$30.GND-, U$31.GND, U$31.GND-, U$4.GND, U$4.GND-, U$41.GND, U$41.GND-, U$42.GND, U$42.GND-, U$43.GND, U$43.GND-, U$44.GND, U$44.GND-, U$45.GND, U$45.GND-, U$46.GND, U$46.GND-, U$47.GND, U$47.GND-, U$48.GND-, U$5.GND, U$5.GND-, U$6.GND, U$6.GND-, U$7.GND, U$7.GND-, U$8.GND, U$8.GND-, U$9.GND, U$9.GND-
- net N$3: now also U$10.VDD, U$10.VDD+, U$11.VDD, U$11.VDD+, U$12.VDD, U$12.VDD+, U$13.VDD, U$13.VDD+, U$14.VDD, U$14.VDD+, U$15.VDD, U$15.VDD+, U$16.VDD, U$16.VDD+, U$17.VDD, U$17.VDD+, U$18.VDD, U$18.VDD+, U$19.VDD, U$19.VDD+, U$2.VDD, U$2.VDD+, U$20.VDD, U$20.VDD+, U$21.VDD, U$21.VDD+, U$22.VDD, U$22.VDD+, U$23.VDD, U$23.VDD+, U$24.VDD, U$24.VDD+, U$25.VDD, U$25.VDD+, U$26.VDD, U$26.VDD+, U$27.VDD, U$27.VDD+, U$28.VDD, U$28.VDD+, U$29.VDD, U$29.VDD+, U$3.VDD, U$3.VDD+, U$30.VDD, U$30.VDD+, U$31.VDD, U$31.VDD+, U$4.VDD, U$4.VDD+, U$41.VDD, U$41.VDD+, U$42.VDD, U$42.VDD+, U$43.VDD, U$43.VDD+, U$44.VDD, U$44.VDD+, U$48.VDD+, U$49.VDD+, U$5.VDD, U$5.VDD+, U$6.VDD, U$6.VDD+, U$7.VDD, U$7.VDD+, U$8.VDD, U$8.VDD+, U$9.VDD, U$9.VDD+
