File: boardpov.sch (EAGLE design)
At the start: 40 parts

Commit message: sdsd
Parts:
- added C1: (no value), adafruit:C-US025-025X050
- added JP1: (no value), pinhead:PINHD-1X3
- added JP2, JP5: (no value), adafruit:PINHD-1X6CB
Connections:
- new net N$1: U$10.GND-, U$11.GND-, U$12.GND-, U$13.GND-, U$14.GND-, U$15.GND-, U$16.GND-, U$17.GND-, U$18.GND-, U$19.GND-, U$2.GND-, U$20.GND-, U$21.GND-, U$22.GND-, U$23.GND-, U$24.GND-, U$25.GND-, U$26.GND-, U$27.GND-, U$28.GND-, U$29.GND-, U$3.GND-, U$30.GND-, U$31.GND-, U$4.GND-, U$41.GND-, U$42.GND-, U$43.GND-, U$44.GND-, U$45.GND-, U$46.GND-, U$47.GND-, U$48.GND-, U$5.GND-, U$6.GND-, U$7.GND-, U$8.GND-, U$9.GND-
- new net N$2: U$1.GND@21, U$48.GND, U$49.GND, U$49.GND-
- new net N$3: U$45.VDD, U$45.VDD+, U$46.VDD, U$46.VDD+, U$47.VDD, U$47.VDD+, U$48.VDD, U$49.VDD
Other:
- moved on the sheet: U$41, U$42, U$43

Commit message: sd
Parts:
- added J1: (no value), SparkFun-Connectors:CONN_02
Connections:
- new net N$10: U$45.CKL, U$46.CK0
- new net N$11: U$45.SD1, U$46.SD0
- new net N$12: U$44.CKL, U$45.CK0
- new net N$13: U$44.SD1, U$45.SD0
- new net N$14: U$26.SD1, U$44.SD0
- new net N$15: U$26.CKL, U$44.CK0
- new net N$16: U$26.SD0, U$27.SD1
- new net N$17: U$26.CK0, U$27.CKL
- new net N$18: U$27.CK0, U$28.CKL
- new net N$19: U$27.SD0, U$28.SD1
- new net N$20: U$28.CK0, U$29.CKL
- new net N$21: U$28.SD0, U$29.SD1
- new net N$22: U$29.CK0, U$30.CKL
- new net N$23: U$29.SD0, U$30.SD1
- new net N$24: U$30.SD0, U$31.SD1
- new net N$25: U$30.CK0, U$31.CKL
- new net N$26: U$25.SD1, U$31.SD0
- new net N$27: U$25.CKL, U$31.CK0
- new net N$28: U$20.CKL, U$21.CK0
- new net N$29: U$20.SD1, U$21.SD0
- new net N$30: U$21.SD1, U$22.SD0
- new net N$31: U$21.CKL, U$22.CK0
- new net N$32: U$22.CKL, U$23.CK0
- new net N$33: U$22.SD1, U$23.SD0
- new net N$34: U$23.SD1, U$24.SD0
- new net N$35: U$23.CKL, U$24.CK0
- new net N$36: U$24.CKL, U$25.CK0
- new net N$37: U$24.SD1, U$25.SD0
- new net N$38: U$14.SD1, U$20.CK0
- new net N$39: U$14.CKL, U$20.SD0
- new net N$4: U$48.SD1, U$49.SD0
- new net N$40: U$14.CK0, U$15.CKL
- new net N$41: U$14.SD0, U$15.SD1
- new net N$42: U$15.CK0, U$16.CKL
- new net N$43: U$15.SD0, U$16.SD1
- new net N$44: U$16.CK0, U$17.CKL
- new net N$45: U$16.SD0, U$17.SD1
- new net N$46: U$17.CK0, U$18.CKL
- new net N$47: U$17.SD0, U$18.SD1
- new net N$48: U$18.CK0, U$19.CKL
- new net N$49: U$18.SD0, U$19.SD1
- new net N$5: U$48.CKL, U$49.CK0
- new net N$50: U$13.SD1, U$19.SD0
- new net N$51: U$13.CKL, U$19.CK0
- new net N$52: U$8.CKL, U$9.CK0
- new net N$53: U$8.SD1, U$9.SD0
- new net N$54: U$10.SD0, U$9.SD1
- new net N$55: U$10.CK0, U$9.CKL
- new net N$56: U$10.CKL, U$11.CK0
- new net N$57: U$10.SD1, U$11.SD0
- new net N$58: U$11.SD1, U$12.SD0
- new net N$59: U$11.CKL, U$12.CK0
- new net N$6: U$47.CKL, U$48.CK0
- new net N$7: U$47.SD1, U$48.SD0
- new net N$8: U$46.SD1, U$47.SD0
- new net N$9: U$46.CKL, U$47.CK0
- net N$1: now also J1.2, U$1.VIN; no longer U$10.GND-, U$11.GND-, U$12.GND-, U$13.GND-, U$14.GND-, U$15.GND-, U$16.GND-, U$17.GND-, U$18.GND-, U$19.GND-, U$2.GND-, U$20.GND-, U$21.GND-, U$22.GND-, U$23.GND-, U$24.GND-, U$25.GND-, U$26.GND-, U$27.GND-, U$28.GND-, U$29.GND-, U$3.GND-, U$30.GND-, U$31.GND-, U$4.GND-, U$41.GND-, U$42.GND-, U$43.GND-, U$44.GND-, U$45.GND-, U$46.GND-, U$47.GND-, U$48.GND-, U$5.GND-, U$6.GND-, U$7.GND-, U$8.GND-, U$9.GND-
- net N$2: now also J1.1, U$1.GND@2, U$10.GND, U$10.GND-, U$11.GND, U$11.GND-, U$12.GND, U$12.GND-, U$13.GND, U$13.GND-, U$14.GND, U$14.GND-, U$15.GND, U$15.GND-, U$16.GND, U$16.GND-, U$17.GND, U$17.GND-, U$18.GND, U$18.GND-, U$19.GND, U$19.GND-, U$2.GND, U$2.GND-, U$20.GND, U$20.GND-, U$21.GND, U$21.GND-, U$22.GND, U$22.GND-, U$23.GND, U$23.GND-, U$24.GND, U$24.GND-, U$25.GND, U$25.GND-, U$26.GND, U$26.GND-, U$27.GND, U$27.GND-, U$28.GND, U$28.GND-, U$29.GND, U$29.GND-, U$3.GND, U$3.GND-, U$30.GND, U$30.GND-, U$31.GND, U$31.GND-, U$4.GND, U$4.GND-, U$41.GND, U$41.GND-, U$42.GND, U$42.GND-, U$43.GND, U$43.GND-, U$44.GND, U$44.GND-, U$45.GND, U$45.GND-, U$46.GND, U$46.GND-, U$47.GND, U$47.GND-, U$48.GND-, U$5.GND, U$5.GND-, U$6.GND, U$6.GND-, U$7.GND, U$7.GND-, U$8.GND, U$8.GND-, U$9.GND, U$9.GND-
- net N$3: now also U$10.VDD, U$10.VDD+, U$11.VDD, U$11.VDD+, U$12.VDD, U$12.VDD+, U$13.VDD, U$13.VDD+, U$14.VDD, U$14.VDD+, U$15.VDD, U$15.VDD+, U$16.VDD, U$16.VDD+, U$17.VDD, U$17.VDD+, U$18.VDD, U$18.VDD+, U$19.VDD, U$19.VDD+, U$2.VDD, U$2.VDD+, U$20.VDD, U$20.VDD+, U$21.VDD, U$21.VDD+, U$22.VDD, U$22.VDD+, U$23.VDD, U$23.VDD+, U$24.VDD, U$24.VDD+, U$25.VDD, U$25.VDD+, U$26.VDD, U$26.VDD+, U$27.VDD, U$27.VDD+, U$28.VDD, U$28.VDD+, U$29.VDD, U$29.VDD+, U$3.VDD, U$3.VDD+, U$30.VDD, U$30.VDD+, U$31.VDD, U$31.VDD+, U$4.VDD, U$4.VDD+, U$41.VDD, U$41.VDD+, U$42.VDD, U$42.VDD+, U$43.VDD, U$43.VDD+, U$44.VDD, U$44.VDD+, U$48.VDD+, U$49.VDD+, U$5.VDD, U$5.VDD+, U$6.VDD, U$6.VDD+, U$7.VDD, U$7.VDD+, U$8.VDD, U$8.VDD+, U$9.VDD, U$9.VDD+
